File: kicad_project/ntaduino.sch (KiCad schematic (older format))
At the start: 22 parts

Commit message: Adding NTAduino real board v0.1
Parts:
- removed C?: 4.7u, symbol CP1
- removed C? (x2): 22p, symbol C
- removed C?: 0.1u, symbol C
- removed D? (x2): 3v6, symbol ZENER
- removed D?: LED, symbol LED
- removed F?: FUSE, symbol FUSE
- removed IC?: ATMEGA8-P, DIL28, symbol ATMEGA8-P
- removed J?: USB, symbol USB
- removed P?: TST, symbol TST
- removed P?: CONNECTOR, symbol CONNECTOR
- removed R? (x2): 100K, symbol R
- removed R?: R, symbol R
- removed R? (x2): 22R, symbol R
- removed X?: 16.000MHz, symbol CRYSTAL
- added C? (x2): 100n, symbol C
- added C?: 1uF, symbol C
- added CON?: USB-MINI-B, symbol USB-MINI-B
- added D?: 1N4148, ~, symbol DIODE
- added D? (x2): 3V6, ~, symbol ZENER
- added D?: LED, ~, symbol LED
- added R? (x2): 10K, symbol R
- added R? (x2): 68, symbol R
- added R?: 2K2, symbol R
- added R?: 1K, symbol R
- added SW?: SW_PUSH, ~, symbol SW_PUSH
Connections:
- net labels removed: CD+, CD-, UD+, UD-
- wire segments 32 -> 35
Other:
- moved on the sheet: C?, IC?, X?

Commit message: populating schematics and associating footprints
Parts:
- removed CON?: USB-MINI-B, symbol USB-MINI-B
- added C5: 100n, symbol C
- added D10, D11: LED3G, ~, symbol LED
- added D12, D13: LED3R++, ~, symbol LED
- added D5: LED-RGB, symbol LED-RGB
- added D6, D7: LED3R, ~, symbol LED
- added D8, D9: LED3Y, ~, symbol LED
- added J1: USB_1, symbol USB_1
- added P1, P2: CONN_14, symbol CONN_14
- added Q1: LTR4206, symbol OPTO_NPN_12
- added R1: 20K, symbol R
- added R11, R12: 10K, symbol R
- added R13, R14, R15, R16, R17, R18, R19, R20, R21: 220, symbol R
- added R22, R23: 150, symbol R
- added R4: 100K, symbol R
- added R5: LDR, symbol R
- added R7: 68, symbol R
- added SP1: SPEAKER, symbol SPEAKER
- added SW2, SW3: SW_PUSH, ~, symbol SW_PUSH
- D1: renamed from D?; value LED -> LED3W
- R6: renamed from R?; value 1K -> 220
- gave numbers to parts that had none: 16
Connections:
- net labels added: P1, P10, P11, P12, P13, P14, P15, P16, P17, P18, P19, P2, P20, P21, P22, P23, P24, P25, P26, P27, P28, P3, P4, P5, P6, P7, P8, P9
- wire segments 35 -> 140
Other:
- note added: "ADC LDR"
- note added: "AREF"
- note added: "Buzzer"
- note added: "HID buttons"
- note added: "LED array"
- note added: "Mode LED"
- note added: "Mode\nSelect"
- note added: "Photo\nreceiver"
- note added: "Photo\ntransmitter"
- moved on the sheet: C1, C2, C3, C4, C6, D1, D2, D3, D4, IC1, R10, R2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

Commit message: preliminary PCB layout with minor schematics changes
Parts:
- added D14: LED3G, ~, symbol LED
- added R24: 330, symbol R
- D1: value LED3W -> LED3R
- D10: value LED3G -> LED3R
- D11: value LED3G -> LED3W
- D6, D7: value LED3R -> LED3G
Connections:
- net +5V: now also R24.1
- net GND: now also D14.2 (K)
- net P11: now also R9.2; no longer R7.2
- net P13: now also R7.2; no longer D4.1 (A)
- net P6: now also D4.1 (A); no longer R9.2
- new net: D14.1 (A), R24.2
Other:
- note removed: "Mode LED"
- moved on the sheet: C1, C2, D1, D10, D11, D5, D6, D7, D8, D9, R13, R14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
