File: kicad_project/ntaduino.sch (KiCad schematic (older format))
At the start: 54 parts, among them IC1 ATMEGA8-P, J1 USB_1, P1 CONN_14, P2 CONN_14, Q1 LTR4206, SW1 SW_PUSH, SW2 SW_PUSH, SW3 SW_PUSH, X1 16.000MHz

Commit message: Rev 1.2
Parts:
- removed D6: LED3G, ~, symbol LED
- removed R16: 220, symbol R
